Commit message: feat: add good visual of boat in gazebo

File: boat_control/urdf/simple_boat.urdf (robot description, URDF)
Before this commit: robot simple_boat, 2 links, 1 joints
Links:
- link base_link: geometry collision box size=0.9 0.42 0.20; visual mesh filename=/home/w1nchie/ros2_ws/src/amr/boat_control/models/benchy.stl scale=0.025 0.025 0.025
